File: lamp_devboard/current_probe.kicad_sch (KiCad schematic)
At the start: 2 parts, among them U301 MAX9938

Commit message: schematics, add battery to power module
Parts:
- U301: footprint (none) -> Package_TO_SOT_SMD:SOT-23-5_HandSoldering
Changed lines of the file:
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@@
       (effects (font (size 1.27 1.27)) (justify left))
     )
-    (property "Footprint" "" (id 2) (at 125.095 96.52 0)
+    (property "Footprint" "Package_TO_SOT_SMD:SOT-23-5_HandSoldering" (id 2) (at 125.095 96.52 0)
       (effects (font (size 1.27 1.27)) hide)
     )
