File: lamp_devboard/io.kicad_sch (KiCad schematic)
At the start: 17 parts, among them SW1001 SW_Push, SW1002 SW_Push, SW1003 SW_Push

Commit message: some changes
Parts:
- removed C1002, C1003: C, Capacitor_SMD:C_0603_1608Metric_Pad1.08x0.95mm_HandSolder, symbol Device:C
- removed D1002: LED_RGB, LED_SMD:LED_WS2812_PLCC6_5.0x5.0mm_P1.6mm, symbol Device:LED_RGB
- removed R1007, R1008, R1009: R, Resistor_SMD:R_0603_1608Metric_Pad0.98x0.95mm_HandSolder, symbol Device:R
- removed SW1002, SW1003: SW_Push, Button_Switch_SMD:SW_Push_1P1T_NO_CK_KMR2, symbol Switch:SW_Push
- added J1001: AudioJack4, Connector_Audio:Jack_3.5mm_CUI_SJ-3524-SMT_Horizontal, symbol Connector:AudioJack4
Connections:
- net GND: now also J1001.T; no longer R1002.2, R1003.2
- net VCC: now also J1001.S
- new net: J1001.R2, R1002.2
- new net: J1001.R1, R1003.2

Commit message: some small changes
Parts:
- removed J1001: AudioJack4, Connector_Audio:Jack_3.5mm_CUI_SJ-3524-SMT_Horizontal, symbol Connector:AudioJack4
- removed R1003: R, Resistor_SMD:R_0603_1608Metric_Pad0.98x0.95mm_HandSolder, symbol Device:R
- added C1002: C, Capacitor_SMD:C_0603_1608Metric_Pad1.08x0.95mm_HandSolder, symbol Device:C
- added D1002: SM6T12A, Diode_SMD:D_SMB, symbol Diode:SM6T12A
- added SW1002: Conn_01x02, Connector_PinHeader_2.54mm:PinHeader_1x02_P2.54mm_Vertical, symbol Connector_Generic:Conn_01x02
Connections:
- net GND: now also R1002.2, D1002.2 (A2)
- net IO_BUTTONS2: now also C1002.2, D1002.1 (A1), SW1002.2 (Pin_2)
- net VCC: now also C1002.1, SW1002.1 (Pin_1)
Other:
- moved on the sheet: R1002
