File: lamp_devboard/lamp_devboard.kicad_pcb (KiCad board)
At the start: 4 copper layers, 40 x 66.8 mm, 110 parts, among them J1001 AudioJack4, J101 Conn_02x02_Counter_Clockwise, J102 Conn_02x02_Counter_Clockwise, J103 Conn_02x02_Counter_Clockwise, J104 Conn_02x02_Counter_Clockwise, J105 Conn_02x02_Counter_Clockwise, J106 Conn_02x02_Counter_Clockwise, J201 Screw_Terminal_01x02, J202 USB_C_Receptacle_USB2.0, J203 Conn_01x03, J901 Conn_02x05_Odd_Even, J905 Conn_01x06, SW1001 SW_Push, U201 TPS212x, U202 BQ24200, U203 FUSB302B01MPX, U204 TLV71318PDBV, U205 TLV71318PDBV, U207 USBLC6-4SC6, U301 MAX9938, U401 TPS63060, U501 MAX9938, U601 TPS63060, U701 MAX9938, U901 STM32L476RG, Y901 Crystal_GND2, Y902 Crystal_GND2

Commit message: some small changes
Parts:
- removed J1001: AudioJack4, Connector_Audio:Jack_3.5mm_CUI_SJ-3524-SMT_Horizontal
- removed R1003: R, Resistor_SMD:R_0603_1608Metric_Pad0.98x0.95mm_HandSolder
- added C1002: C, Capacitor_SMD:C_0603_1608Metric_Pad1.08x0.95mm_HandSolder, B.Cu at (44.5, 97.3)
- added D1002: SM6T12A, Diode_SMD:D_SMB, B.Cu at (42.4, 89.1)
- added SW1002: Conn_01x02, Connector_PinHeader_2.54mm:PinHeader_1x02_P2.54mm_Vertical, F.Cu at (42.4, 98.9)
- J201: value Screw_Terminal_01x02 -> Conn_02x02_Counter_Clockwise; footprint TerminalBlock:TerminalBlock_bornier-2_P5.08mm -> Connector_PinSocket_2.54mm:PinSocket_2x02_P2.54mm_Vertical
- moved R1002 60.6 mm to (43.3, 93.6)
- moved J905 7.75 mm to (84.4, 83.2)
- moved J201 3.56 mm to (46.5, 96.3), turned to 90 degrees
Connections:
- J201 pad 2: /power_in/TerminalPIn_ -> GND
- J905 pad 1: Net-(J905-Pad1) -> /1V8_D
- J905 pad 2: Net-(J905-Pad2) -> GND
- R1002 pad 2: Net-(J1001-PadR2) -> GND
- U901 pad 28: Net-(J905-Pad1) -> unconnected-(U901-Pad28)
- U901 pad 29: Net-(J905-Pad5) -> unconnected-(U901-Pad29)
- U901 pad 30: Net-(J905-Pad6) -> unconnected-(U901-Pad30)
- U901 pad 33: unconnected-(U901-Pad33) -> (no net)
- U901 pad 34: unconnected-(U901-Pad34) -> (no net)
- U901 pad 41: /uC/UC_BUTTONS1 -> /io/IO_BUTTONS1
- U901 pad 42: /uC/UC_BUTTONS2 -> /io/IO_BUTTONS2
- U901 pad 51: unconnected-(U901-Pad51) -> Net-(J905-Pad3)
- U901 pad 52: unconnected-(U901-Pad52) -> Net-(J905-Pad4)
- U901 pad 53: unconnected-(U901-Pad53) -> Net-(J905-Pad5)
- U901 pad 57: Net-(J905-Pad2) -> Net-(J905-Pad6)
- U901 pad 61: Net-(J905-Pad3) -> unconnected-(U901-Pad61)
- U901 pad 62: Net-(J905-Pad4) -> unconnected-(U901-Pad62)
Routing:
- net /io/IO_BUTTONS2: track 0.00 -> 39.1 mm, vias 0 -> 1
- net /1V8_D: track 83.9 -> 108.6 mm
- net unconnected-(U901-Pad51): track 24.6 -> 0.00 mm
- net Net-(J905-Pad3): track 0.00 -> 24.6 mm
- net unconnected-(U901-Pad52): track 23.3 -> 0.00 mm
- net Net-(J905-Pad4): track 0.00 -> 23.3 mm
- net unconnected-(U901-Pad53): track 22.1 -> 0.00 mm, vias 1 -> 0
- net Net-(J905-Pad5): track 0.00 -> 22.1 mm, vias 0 -> 1
- net Net-(J905-Pad6): track 0.00 -> 18.4 mm, vias 0 -> 1
- net Net-(J905-Pad2): track 18.4 -> 0.00 mm, vias 1 -> 0
- net GND: track 111.9 -> 125.5 mm, vias 63 -> 65
- net /power_in/Pout_: track 20.6 -> 24.0 mm

Commit message: first version of the pcb board
Parts:
- removed Le101, Le102: Lense, lamp_devboard_lib:EMILY
- added R402: R, Resistor_SMD:R_0603_1608Metric_Pad0.98x0.95mm_HandSolder, F.Cu at (71.8, 76.5)
- added R602: R, Resistor_SMD:R_0603_1608Metric_Pad0.98x0.95mm_HandSolder, F.Cu at (52.9, 76.7)
- added TP101: TestPoint, TestPoint:TestPoint_Pad_1.0x1.0mm, F.Cu at (72.3, 33.6)
- added TP102: TestPoint, TestPoint:TestPoint_Pad_1.0x1.0mm, F.Cu at (47.7, 33.4)
- HS101, HS102, J102, J104, J106: moved to B.Cu
- J201: footprint Connector_PinSocket_2.54mm:PinSocket_2x02_P2.54mm_Vertical -> Connector_PinHeader_2.54mm:PinHeader_2x02_P2.54mm_Vertical
- J202: footprint Connector_USB:USB_C_Receptacle_Amphenol_12401548E4-2A -> lamp_devboard_lib:AMPHENOL_124018312112A
- moved TH102 96.8 mm to (55.5, 33.6), turned to 90 degrees
- moved HS101 79.3 mm to (68.5, 33.5), turned to 180 degrees
- moved J102 74.5 mm to (78.3, 34.8), turned to 90 degrees
- moved HS102 67.2 mm to (51.5, 33.6), turned to 180 degrees
- moved J104 65.4 mm to (58.7, 32.2), turned to -90 degrees
- moved TH101 61.3 mm to (64.5, 33.5), turned to 90 degrees
- moved D101 57.1 mm to (68.5, 33.5), turned to 90 degrees
- moved J106 54.8 mm to (44.2, 34.8), turned to 90 degrees
- moved D102 52.5 mm to (51.5, 33.5), turned to 90 degrees
- moved J202 21.9 mm to (70.8, 117.3)
- moved C1001 18.4 mm to (63.5, 77.2), turned to 90 degrees
- moved C901 18.4 mm to (58.0, 93.1)
- moved J201 18.3 mm to (49.1, 114.4), turned to -90 degrees
- moved C1002 18.1 mm to (44.5, 115.4)
- moved C201 18.1 mm to (46.1, 104.2)
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Connections:
- D101 pad 1: GND -> GND1
- D101 pad 2: /current_probe_1/IV_Iout -> /LED1_Pin
- D102 pad 1: GND -> GND2
- D102 pad 2: /current_probe_2/IV_Iout -> /LED2_Pin
- J102 pad 1: GND -> GND1
- J102 pad 2: GND -> GND1
- J102 pad 3: /current_probe_1/IV_Iout -> /LED1_Pin
- J102 pad 4: /current_probe_1/IV_Iout -> /LED1_Pin
- J106 pad 1: GND -> GND2
- J106 pad 2: GND -> GND2
- J106 pad 3: /current_probe_2/IV_Iout -> /LED2_Pin
- J106 pad 4: /current_probe_2/IV_Iout -> /LED2_Pin
Routing:
- net /1V8_D: track 108.6 -> 128.7 mm
- net GND: track 125.5 -> 139.3 mm, vias 65 -> 69
- net Net-(J202-PadA5): track 29.5 -> 16.3 mm
- net Net-(J905-Pad4): track 23.3 -> 35.2 mm
- net Net-(J905-Pad6): track 18.4 -> 27.5 mm
- net /power_in/UsbPIn: track 10.7 -> 17.0 mm, vias 4 -> 6
- net Net-(J202-PadB5): track 12.8 -> 17.9 mm, vias 0 -> 1
- net Net-(J905-Pad5): track 22.1 -> 26.9 mm
- net /current_probe_in/IV_Iout: track 0.00 -> 4.71 mm
- net Net-(J905-Pad3): track 24.6 -> 29.1 mm
- net /current_probe_1/IV_Out: track 28.6 -> 24.4 mm, vias 0 -> 2
- net Net-(J104-Pad4): track 0.00 -> 3.73 mm
- net Net-(J104-Pad2): track 0.00 -> 3.55 mm
- net Net-(J104-Pad1): track 0.00 -> 3.41 mm
- net Net-(J104-Pad3): track 0.00 -> 3.35 mm
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- added copper zone on F.Cu, net /LED1_Pin
- added copper zone on F.Cu, net /LED2_Pin
- added copper zone on F.Cu, net GND1
- added copper zone on F.Cu, net GND2
- added copper zone on F.Cu, net Net-(D101-Pad3)
- added copper zone on F.Cu, net Net-(D102-Pad3)
Other:
- board size 40 x 66.8 mm -> 48.6 x 94.9 mm
