File: lamp_devboard/power_in.kicad_sch (KiCad schematic)
At the start: 35 parts, among them J201 Conn_02x02_Counter_Clockwise, J202 USB_C_Receptacle_USB2.0, J203 Conn_01x03, U201 TPS212x, U202 BQ24200, U203 FUSB302B01MPX, U204 TLV71318PDBV, U205 TLV71318PDBV, U207 USBLC6-4SC6

Commit message: first version of the pcb board
Parts:
- J201: footprint Connector_PinSocket_2.54mm:PinSocket_2x02_P2.54mm_Vertical -> Connector_PinHeader_2.54mm:PinHeader_2x02_P2.54mm_Vertical
- J202: footprint Connector_USB:USB_C_Receptacle_Amphenol_12401548E4-2A -> lamp_devboard_lib:AMPHENOL_124018312112A
Changed lines of the file:
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@@
   (junction (at 77.47 38.735) (diameter 0) (color 0 0 0 0)
-  )
-  (junction (at 42.545 212.09) (diameter 0) (color 0 0 0 0)
   )
   (junction (at 73.66 199.39) (diameter 0) (color 0 0 0 0)
@@
     (stroke (width 0) (type default) (color 0 0 0 0))
   )
-  (wire (pts (xy 41.91 212.09) (xy 42.545 212.09))
-    (stroke (width 0) (type default) (color 0 0 0 0))
-  )
   (bus (pts (xy 125.095 137.16) (xy 128.27 137.16))
     (stroke (width 0) (type default) (color 0 0 0 0))
@@
     (property "Reference" "J202" (id 0) (at 38.1 30.48 0))
     (property "Value" "USB_C_Receptacle_USB2.0" (id 1) (at 38.1 33.02 0))
-    (property "Footprint" "Connector_USB:USB_C_Receptacle_Amphenol_12401548E4-2A" (id 2) (at 41.91 53.975 0)
+    (property "Footprint" "lamp_devboard_lib:AMPHENOL_124018312112A" (id 2) (at 41.91 53.975 0)
       (effects (font (size 1.27 1.27)) hide)
     )
@@
       (effects (font (size 1.27 1.27)) (justify right) hide)
     )
-    (property "Footprint" "Connector_PinSocket_2.54mm:PinSocket_2x02_P2.54mm_Vertical" (id 2) (at 42.545 207.01 0)
-      (effects (font (size 1.27 1.27)) hide)
-    )
+    (property "Footprint" "Connector_PinHeader_2.54mm:PinHeader_2x02_P2.54mm_Vertical" (id 2) (at 42.545 207.01 0)
+      (effects (font (size 1.27 1.27)) hide)
+    )
